Commit message: updated

File: src/rby1_urdf_visualization/urdf/rby1_urdf/model.urdf (robot description, URDF)
Before this commit: robot RB_Y1_V1.0.1, 34 links, 33 joints
Links:
- added link link_zvid, mass 0.03585374; visual mesh filename=package://rby1_urdf_visualization/urdf/rby1_urdf/meshes/zvi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 scale=0.1 0.1 0.1
Joints:
- added joint zvid: type fixed, parent link_head_2, child link_zvid, origin xyz=0.022 0.0 0.04 rpy=-1.5708 0.0 1.5708, axis 0 0 0

Commit message: update all

File: src/rby1_urdf_visualization/urdf/rby1_urdf/model.urdf (robot description, URDF)
Before this commit: robot RB_Y1_V1.0.1, 35 links, 34 joints
Joints:
- joint zvid: origin xyz=0.022 0.0 0.04 rpy=-1.5708 0.0 1.5708 -> xyz=0.0 0.0 0.04 rpy=-1.5708 0.0 1.5708

Commit message: updteed

File: src/rby1_urdf_visualization/urdf/rby1_urdf/model.urdf (robot description, URDF)
Before this commit: robot RB_Y1_V1.0.1, 35 links, 34 joints
Links:
- added link link_camera_frame, mass 0.03585374; visual cylinder length=0.01 radius=0.01
Joints:
- added joint camera_frame: type fixed, parent link_zvid, child link_camera_frame, origin xyz=0.07702 -0.039419 -0.0250 rpy=0.0 3.20372871 0.0, axis 0 0 0
